File: stusb1602-breakout/stusb1602-breakout.kicad_sch (KiCad schematic)
At the start: 4 parts

Commit message: added stusb
Parts:
- added U1: STUSB1602AQTR, QFN50P400X400X100-25N, symbol STUSB1602AQTR:STUSB1602AQTR
Changed lines of the file:
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@@
+		)
+	)
+	(symbol
+		(lib_id "STUSB1602AQTR:STUSB1602AQTR")
+		(at 162.56 59.69 0)
+		(unit 1)
+		(exclude_from_sim no)
+		(in_bom yes)
+		(on_board yes)
+		(dnp no)
+		(fields_autoplaced yes)
+		(property "Reference" "U1"
+			(at 162.56 31.75 0)
+			(effects
+				(font
+					(size 1.27 1.27)
+				)
+			)
+		)
+		(property "Value" "STUSB1602AQTR"
+			(at 162.56 34.29 0)
+			(effects
+				(font
+					(size 1.27 1.27)
+				)
+			)
+		)
+		(property "Footprint" "QFN50P400X400X100-25N"
+			(at 162.56 59.69 0)
+			(effects
+				(font
+					(size 1.27 1.27)
+				)
+				(justify bottom)
+				(hide yes)
+			)
+		)
+		(property "Datasheet" ""
+			(at 162.56 59.69 0)
+			(effects
+				(font
+					(size 1.27 1.27)
+				)
+				(hide yes)
+			)
+		)
+		(property "Description" ""
+			(at 162.56 59.69 0)
+			(effects
+				(font
+					(size 1.27 1.27)
+				)
+				(hide yes)
+			)
+		)
+		(property "MF" "STMicroelectronics"
+			(at 162.56 59.69 0)
+			(effects
+				(font
+					(size 1.27 1.27)
+				)
+				(justify bottom)
+				(hide yes)
+			)
+		)
+		(property "Description_1" "\n                        \n                            USB, Type-C Controller PMIC 24-QFN-EP (4x4)\n                        \n"
+			(at 162.56 59.69 0)
+			(effects
+				(font
+					(size 1.27 1.27)
+				)
+				(justify bottom)
+				(hide yes)
+			)
+		)
+		(property "Package" "VQFN-24 STMicroelectronics"
+			(at 162.56 59.69 0)
+			(effects
+				(font
+					(size 1.27 1.27)
+				)
+				(justify bottom)
+				(hide yes)
+			)
+		)
+		(property "Price" "None"
+			(at 162.56 59.69 0)
+			(effects
+				(font
+					(size 1.27 1.27)
+				)
+				(justify bottom)
+				(hide yes)
+			)
+		)
+		(property "Check_prices" "https://www.snapeda.com/parts/STUSB1602AQTR/STMicroelectronics/view-part/?ref=eda"
+			(at 162.56 59.69 0)
+			(effects
+				(font
+					(size 1.27 1.27)
+				)
+				(justify bottom)
+				(hide yes)
+			)
+		)
+		(property "PART_REV" "3"
+			(at 162.56 59.69 0)
+			(effects
+				(font
+					(size 1.27 1.27)
+				)
+				(justify bottom)
+				(hide yes)
+			)
+		)
+		(property "STANDARD" "IPC-7351B"
+			(at 162.56 59.69 0)
+			(effects
+				(font
+					(size 1.27 1.27)
+				)
+				(justify bottom)
+				(hide yes)
+			)
+		)
+		(property "SnapEDA_Link" "https://www.snapeda.com/parts/STUSB1602AQTR/STMicroelectronics/view-part/?ref=snap"
+			(at 162.56 59.69 0)
+			(effects
+				(font
+					(size 1.27 1.27)
+				)
+				(justify bottom)
+				(hide yes)
+			)
+		)
+		(property "MP" "STUSB1602AQTR"
+			(at 162.56 59.69 0)
+			(effects
+				(font
+					(size 1.27 1.27)
+				)
+				(justify bottom)
+				(hide yes)
+			)
+		)
+		(property "Availability" "In Stock"
+			(at 162.56 59.69 0)
+			(effects
+				(font
+					(size 1.27 1.27)
+				)
+				(justify bottom)
+				(hide yes)
+			)
+		)
+		(property "MANUFACTURER" "ST Microelectronics"
+			(at 162.56 59.69 0)
+			(effects
+				(font
+					(size 1.27 1.27)
+				)
+				(justify bottom)
+				(hide yes)
+			)
+		)
+		(pin "2"
+		)
+		(pin "9"
+		)
+		(pin "23"
+		)
+		(pin "17"
+		)
+		(pin "12"
+		)
+		(pin "7"
+		)
+		(pin "11"
+		)
+		(pin "18"
+		)
+		(pin "1"
+		)
+		(pin "22"
+		)
+		(pin "24"
+		)
+		(pin "5"
+		)
+		(pin "25"
+		)
+		(pin "4"
+		)
+		(pin "16"
+		)
+		(pin "13"
+		)
+		(pin "14"
+		)
+		(pin "15"
+		)
+		(pin "19"
+		)
+		(pin "21"
+		)
+		(pin "8"
+		)
+		(pin "20"
+		)
+		(pin "10"
+		)
+		(pin "3"
+		)
+		(pin "6"
+		)
+		(instances
+			(project ""
+				(path "/9c1e018e-4236-4221-bb76-4e952826dafd"
+					(reference "U1")
+					(unit 1)
+				)
+			)
 		)
 	)

Commit message: schematic progress
Parts:
- removed C1: 1μF, Capacitor_SMD:C_0603_1608Metric, symbol Device:C
- removed C2: 10μF, Capacitor_SMD:C_0603_1608Metric, symbol Device:C
- removed R1: 10K, Resistor_SMD:R_0603_1608Metric, symbol Device:R_US
- removed R2: 1K, Resistor_SMD:R_0603_1608Metric, symbol Device:R_US
- added C1, C3, C5: 1μF, Capacitor_SMD:C_0603_1608Metric, symbol Device:C_Small
- added C4: 10μF, Capacitor_SMD:C_0603_1608Metric, symbol Device:C_Small
- added R1, R2: 1K, Resistor_SMD:R_0603_1608Metric, symbol Device:R_Small_US
- added R10, R3, R4, R5, R6, R7, R8, R9: 10K, Resistor_SMD:R_0603_1608Metric, symbol Device:R_Small_US
Connections:
- net at U1.1 (CC1DB): now also U1.2 (CC1)
- net GND: now reaches U1.10 (GND)
- net GND: now also U1.13 (ADDR0), U1.25 (EP(GND)), C1.2, C3.1, C4.2, C5.2, R1.2, R2.2
- net at U1.11 (MOSI): now also R10.2
- net at U1.12 (NSS): now also R8.2
- net at U1.14 (MISO): now also R7.2
- net at U1.15 (TX_EN): now also R2.1
- net at U1.16 (SCLK): now also R9.2
- net at U1.17 (A_B_SIDE): now also R3.2
- net at U1.21 (VREG_1V2): now also C3.2
- net +3V3: now reaches U1.22 (VSYS)
- net +3V3: now also C1.1, R10.1, R3.1, R4.1, R5.1, R6.1, R7.1, R8.1, R9.1
- net at U1.23 (VREG_2V7): now also C5.1
- net +5V: now reaches U1.3 (VCONN)
- net +5V: now also C4.1
- net at U1.4 (CC2): now also U1.5 (CC2DB)
- net at U1.6 (RESET): now also R1.1
- net at U1.7 (SCL): now also R4.2
- net at U1.8 (SDA): now also R5.2
- net at U1.9 (~{ALERT}): now also R6.2
